Commit message: 融入仿真的功能包

File: src/scout_ros/scout_description/urdf/scout_mini.urdf.xacro (robot description, xacro)
@@ -15,4 +15,13 @@
     <xacro:property name="wheel_length" value="0.8e-01" />
     <xacro:property name="wheel_radius" value="1.600e-01" />
+    <xacro:property name="frame_length" value="0.35" />
+    <xacro:property name="frame_width" value="0.27" />
+    <xacro:property name="frame_height" value="0.14" />
+    <xacro:property name="frame_profile" value="0.04" />
+    <xacro:property name="frame_z_offset" value="-0.05" />
+    <material name="aluminum">
+        <color rgba="0.7 0.7 0.7 1" />
+    </material>
+    <xacro:include filename="$(find sick_safetyscanners_description)/urdf/nanoscan3.urdf.xacro" />
     <!-- Base link -->
     <link name="base_link">
@@ -53,8 +62,8 @@
         <origin xyz="${wheelbase/2} ${-track/2} ${wheel_vertical_offset}" rpy="1.57 0 0" />
     </xacro:scout_mini_wheel>
-    <xacro:scout_mini_wheel wheel_prefix="front_left">
+    <xacro:scout_mini_wheel wheel_prefix="front_left" axis_sign="1">
         <origin xyz="${wheelbase/2} ${track/2} ${wheel_vertical_offset}" rpy="-1.57 0 0" />
     </xacro:scout_mini_wheel>
-    <xacro:scout_mini_wheel wheel_prefix="rear_left">
+    <xacro:scout_mini_wheel wheel_prefix="rear_left" axis_sign="1">
         <origin xyz="${-wheelbase/2} ${track/2} ${wheel_vertical_offset}" rpy="-1.57 0 0" />
     </xacro:scout_mini_wheel>
@@ -74,4 +83,74 @@
         <child link="rear_mount" />
     </joint>
+    <!-- Aluminum frame (40x40) -->
+    <joint name="frame_joint" type="fixed">
+        <origin xyz="0 0 ${base_z_size/2 + frame_z_offset}" rpy="0 0 0" />
+        <parent link="base_link" />
+        <child link="frame_link" />
+    </joint>
+    <link name="frame_link">
+        <!-- Vertical posts -->
+        <visual>
+            <origin xyz="${frame_length/2 - frame_profile/2} ${frame_width/2 - frame_profile/2} ${frame_height/2}" rpy="0 0 0" />
+            <geometry>
+                <box size="${frame_profile} ${frame_profile} ${frame_height}" />
+            </geometry>
+            <material name="aluminum" />
+        </visual>
+        <visual>
+            <origin xyz="${frame_length/2 - frame_profile/2} ${-(frame_width/2 - frame_profile/2)} ${frame_height/2}" rpy="0 0 0" />
+            <geometry>
+                <box size="${frame_profile} ${frame_profile} ${frame_height}" />
+            </geometry>
+            <material name="aluminum" />
+        </visual>
+        <visual>
+            <origin xyz="${-(frame_length/2 - frame_profile/2)} ${frame_width/2 - frame_profile/2} ${frame_height/2}" rpy="0 0 0" />
+            <geometry>
+                <box size="${frame_profile} ${frame_profile} ${frame_height}" />
+            </geometry>
+            <material name="aluminum" />
+        </visual>
+        <visual>
+            <origin xyz="${-(frame_length/2 - frame_profile/2)} ${-(frame_width/2 - frame_profile/2)} ${frame_height/2}" rpy="0 0 0" />
+            <geometry>
+                <box size="${frame_profile} ${frame_profile} ${frame_height}" />
+            </geometry>
+            <material name="aluminum" />
+        </visual>
+        <!-- Top perimeter (4 bars) -->
+        <visual>
+            <origin xyz="0 ${frame_width/2 - frame_profile/2} ${frame_height - frame_profile/2}" rpy="0 0 0" />
+            <geometry>
+                <box size="${frame_length - 2*frame_profile} ${frame_profile} ${frame_profile}" />
+            </geometry>
+            <material name="aluminum" />
+        </visual>
+        <visual>
+            <origin xyz="0 ${-(frame_width/2 - frame_profile/2)} ${frame_height - frame_profile/2}" rpy="0 0 0" />
+            <geometry>
+                <box size="${frame_length - 2*frame_profile} ${frame_profile} ${frame_profile}" />
+            </geometry>
+            <material name="aluminum" />
+        </visual>
+        <visual>
+            <origin xyz="${frame_length/2 - frame_profile/2} 0 ${frame_height - frame_profile/2}" rpy="0 0 0" />
+            <geometry>
+                <box size="${frame_profile} ${frame_width - 2*frame_profile} ${frame_profile}" />
+            </geometry>
+            <material name="aluminum" />
+        </visual>
+        <visual>
+            <origin xyz="${-(frame_length/2 - frame_profile/2)} 0 ${frame_height - frame_profile/2}" rpy="0 0 0" />
+            <geometry>
+                <box size="${frame_profile} ${frame_width - 2*frame_profile} ${frame_profile}" />
+            </geometry>
+            <material name="aluminum" />
+        </visual>
+    </link>
+    <!-- NanoScan3 2D激光雷达 -->
+    <xacro:nanoscan3 prefix="nano" parent_link="base_link" topic="/scan" robot_namespace="$(arg robot_namespace)">
+        <origin xyz="0.13 -0.045 ${base_z_size/2 + frame_height + frame_z_offset}" rpy="0 0 1.57079632679"/>
+    </xacro:nanoscan3>
     <!-- Additional definitions -->
     <xacro:include filename="$(arg urdf_extras)" />

File: src/scout_ros/scout_description/urdf/scout_mini_wheel.xacro (robot description, xacro)
@@ -1,5 +1,5 @@
 <?xml version="1.0"?>
 <robot xmlns:xacro="http://ros.org/wiki/xacro" name="scout_wheel">
-    <xacro:macro name="scout_mini_wheel" params="wheel_prefix *joint_pose">
+    <xacro:macro name="scout_mini_wheel" params="wheel_prefix axis_sign:=-1 *joint_pose">
         <link name="${wheel_prefix}_wheel_link">
             <inertial>
@@ -28,5 +28,5 @@
             <child link="${wheel_prefix}_wheel_link"/>
             <xacro:insert_block name="joint_pose"/>
-            <axis xyz="0 0 -1" rpy="0 0 0" />
+            <axis xyz="0 0 ${axis_sign}" rpy="0 0 0" />
         </joint>
     </xacro:macro>

Commit message: 添加完成仿真

File: src/scout_ros/scout_description/urdf/scout_mini.urdf.xacro (robot description, xacro)
@@ -21,5 +21,5 @@
     <xacro:property name="frame_z_offset" value="-0.05" />
     <material name="aluminum">
-        <color rgba="0.7 0.7 0.7 1" />
+        <color rgba="0 0 0 1" />
     </material>
     <xacro:include filename="$(find sick_safetyscanners_description)/urdf/nanoscan3.urdf.xacro" />

File: src/sick_safetyscanners_description/urdf/nanoscan3.urdf.xacro (robot description, xacro)
@@ -12,6 +12,6 @@
         </geometry>
         <origin xyz="0 0 0.051" rpy="1.5707963267948966 0 -1.5707963267948966" />
-        <material name="sick_yellow">
-          <color rgba="1 1 0 1" />
+        <material name="sick_gray">
+          <color rgba="0.5 0.5 0.5 1" />
         </material>
       </visual>

Commit message: Add Gazebo IMU and sim validation scripts

File: src/scout_ros/scout_description/urdf/scout_mini.urdf.xacro (robot description, xacro)
@@ -55,4 +55,24 @@
         <parent link="base_link" />
         <child link="inertial_link" />
+    </joint>
+    <!-- IMU frame: match the real scout_imu_with_tf.launch coarse mounting pose. -->
+    <link name="imu_link">
+        <inertial>
+            <mass value="0.01" />
+            <origin xyz="0 0 0" />
+            <inertia ixx="1e-6" ixy="0" ixz="0" iyy="1e-6" iyz="0" izz="1e-6" />
+        </inertial>
+        <visual>
+            <origin xyz="0 0 0" rpy="0 0 0" />
+            <geometry>
+                <box size="0.03 0.03 0.01" />
+            </geometry>
+            <material name="aluminum" />
+        </visual>
+    </link>
+    <joint name="base_to_imu_joint" type="fixed">
+        <origin xyz="0.10 -0.045 0.0" rpy="0 0 0" />
+        <parent link="base_link" />
+        <child link="imu_link" />
     </joint>
     <!-- Scout wheel macros -->
