Commit message: 修复仿真四轮 skid-steer 接触参数(A 步) 并完成 B+C bisect
背景:
官方 AgileX Scout Mini Gazebo 模型存在多处接触建模缺陷,导致仿真原地自转
中心系统性漂移 21cm + 高频抖动,且 sim-real 轨迹跟踪差距明显。为 anti-slosh
MPC 验证与后续 RL 训练做 sim 底座准备,定位并按 ROI 顺序修复。

A 步(已生效):
在本仓库 bridge 侧 extras xacro 给四个 wheel_link 注入 ODE 接触参数,
覆盖 official scout_mini.gazebo 被整段注释掉的全局摩擦/接触块以及
scout_mini_wheel.gazebo 只有 transmission 没有 reference 块的问题。
参数(v2 调优,首版 kd=100 因 ringing 已撤回):
  mu1=1.0 mu2=0.5 fdir1="1 0 0" minDepth=0.001 maxContacts=64
不修改 /data/a/official_scout_ws,只动本仓库 extras 文件。
spin test 验证 pose drift peak 从 0.217m 降到 0.116m(降 47%,目标 50%)。

B/C bisect(已回退):
fork mini_abs.xacro / scout_mini.gazebo 试图同时修两个剩余问题:
  B = 去掉右轮 wheel_vertical_offset + 0.001 偏置(四轮共面)
  C = skid_steer 插件 torque 1000 -> 50 (压实物峰值量级)
四组对比(同 before bag 基线):
  A 单独    pose drop +47% (最好)
  ab       pose drop -14% (反而变差)
  ac       pose drop +8%
  abc      pose drop +4%
归因:upstream 的 +0.001 大概率是故意打破 4 点共面以规避 ODE 接触过约束;
torque=50 在原地自转工况下 fmax 不足以让 ODE 速度约束跟上目标,
轮速跟踪误差累积反而放大漂移。
bisect 后 launch 切回 upstream mini_abs.xacro 与 torque=1000,
两个 fork 文件保留在仓库但未被引用,作为未来 D(惯量)或对角偏置实验的
基础设施;若要彻底清理直接 rm 即可。

工具:
record_spin_test.sh - 对同一 spawn 位姿录纯角速度自转 bag(30s,0.2 rad/s),
                      自动 /gazebo/set_model_state 复位 + 写 meta.json。
analysis/analyze_spin_test.py - 对比 before/after bag, 输出 pose drift
                                peak/RMS, IMU 5-20Hz 谱能量, PASS/FAIL。

文档:
docs/Claude/修改方案-时间-简介/2026-05-19_仿真skid-steer接触模型修复方案.md
  完整缺陷清单(A-F),修复路线,fork 策略,后续 D 与 cmd_vel ramp 占位。
docs/Claude/修改日志-时间/2026-05-19.md
  追加 A v1/v2 实验、B+C 应用、abc/ab/ac bisect 全部数据与诊断、
  回退操作与可回退命令。

可回退:
  git checkout -- src/scout_ros/scout_description/urdf/official_scout_mini_imu_extras.urdf.xacro
  git checkout -- src/scout_ros/scout_description/launch/scout_mini_stock_abs_imu.launch
  rm src/scout_ros/scout_description/urdf/mini_abs_fixed.xacro
  rm src/scout_ros/scout_description/urdf/scout_mini_fixed.gazebo

Co-Authored-By: Claude Opus 4.7 <noreply@anthropic.com>

File: src/scout_ros/scout_description/urdf/official_scout_mini_imu_extras.urdf.xacro (robot description, xacro)
@@ -52,3 +52,24 @@
     </plugin>
   </gazebo>
+  <!-- Wheel contact parameters (fix A from 2026-05-19_仿真skid-steer接触模型修复方案):
+       official scout_mini.gazebo 把全局摩擦块整段注释掉,scout_mini_wheel.gazebo
+       也只有 <transmission>,导致四个轮子走 Gazebo 默认 mu1=mu2=1 各向同性摩擦,
+       是 stick-slip + 原地自转抖动的头号原因。这里补上 4 个 wheel_link 的接触参数。
+       fdir1 在各 wheel_link 局部坐标系下都是 x 方向(滚动方向),因为 cylinder 沿 z 轴。 -->
+  <!-- v2 (2026-05-19 iteration after first try made 5-20Hz energy +275%):
+       v1 用 kd=100 + mu2=0.3 + maxVel=1.0,造成接触阻尼 ringing。
+       v2 移除 kp/kd/maxVel,回到 ODE 默认刚体接触;mu2 提到 0.5。 -->
+  <xacro:macro name="scout_wheel_contact" params="wheel_prefix">
+    <gazebo reference="${wheel_prefix}_wheel_link">
+      <mu1>1.0</mu1>
+      <mu2>0.5</mu2>
+      <fdir1>1 0 0</fdir1>
+      <minDepth>0.001</minDepth>
+      <maxContacts>64</maxContacts>
+    </gazebo>
+  </xacro:macro>
+  <xacro:scout_wheel_contact wheel_prefix="front_left" />
+  <xacro:scout_wheel_contact wheel_prefix="front_right" />
+  <xacro:scout_wheel_contact wheel_prefix="rear_left" />
+  <xacro:scout_wheel_contact wheel_prefix="rear_right" />
 </robot>
